File: Test.sch (EAGLE design)
At the start: 1 part

Commit message: [add]とりあえず書いてみた
Parts:
- added C1, C2, C3, C4: (no value), capacitor-wima:C2.5/2
- added R1, R2, R3, R4: (no value), resistor-power:RAC01
Connections:
- new net +5V: R3.2, R4.2
- new net GND: C2.2, C3.2, C4.2, U$1.VSS
- new net N$1: C2.1, U$1.GND
- new net N$2: C3.1, R3.1, U$1.CKIN
- new net N$3: C1.2, R1.1, R2.1
- new net N$4: C1.1, U$1.IN
- new net N$5: C4.1, R4.1, U$1.VDD
Changed lines of the file:
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@@
 <parts>
 <part name="U$1" library="ynakano1127" deviceset="MSGEQ7" device=""/>
+<part name="P+1" library="supply1" library_urn="urn:adsk.eagle:library:371" deviceset="+5V" device=""/>
+<part name="C1" library="capacitor-wima" library_urn="urn:adsk.eagle:library:116" deviceset="C" device="2.5/2" package3d_urn="urn:adsk.eagle:package:5415/1"/>
+<part name="C2" library="capacitor-wima" library_urn="urn:adsk.eagle:library:116" deviceset="C" device="2.5/2" package3d_urn="urn:adsk.eagle:package:5415/1"/>
+<part name="C3" library="capacitor-wima" library_urn="urn:adsk.eagle:library:116" deviceset="C" device="2.5/2" package3d_urn="urn:adsk.eagle:package:5415/1"/>
+<part name="R1" library="resistor-power" library_urn="urn:adsk.eagle:library:344" deviceset="R" device="AC01" package3d_urn="urn:adsk.eagle:package:25124/1"/>
+<part name="R2" library="resistor-power" library_urn="urn:adsk.eagle:library:344" deviceset="R" device="AC01" package3d_urn="urn:adsk.eagle:package:25124/1"/>
+<part name="R3" library="resistor-power" library_urn="urn:adsk.eagle:library:344" deviceset="R" device="AC01" package3d_urn="urn:adsk.eagle:package:25124/1"/>
+<part name="P+2" library="supply1" library_urn="urn:adsk.eagle:library:371" deviceset="+5V" device=""/>
+<part name="GND1" library="supply1" library_urn="urn:adsk.eagle:library:371" deviceset="GND" device=""/>
+<part name="GND2" library="supply1" library_urn="urn:adsk.eagle:library:371" deviceset="GND" device=""/>
+<part name="GND3" library="supply1" library_urn="urn:adsk.eagle:library:371" deviceset="GND" device=""/>
+<part name="GND4" library="supply1" library_urn="urn:adsk.eagle:library:371" deviceset="GND" device=""/>
+<part name="C4" library="capacitor-wima" library_urn="urn:adsk.eagle:library:116" deviceset="C" device="2.5/2" package3d_urn="urn:adsk.eagle:package:5415/1"/>
+<part name="R4" library="resistor-power" library_urn="urn:adsk.eagle:library:344" deviceset="R" device="AC01" package3d_urn="urn:adsk.eagle:package:25124/1"/>
+<part name="P+3" library="supply1" library_urn="urn:adsk.eagle:library:371" deviceset="+5V" device=""/>
+<part name="GND5" library="supply1" library_urn="urn:adsk.eagle:library:371" deviceset="GND" device=""/>
 </parts>
 <sheets>
@@
 <instances>
 <instance part="U$1" gate="G$1" x="0" y="0" smashed="yes"/>
+<instance part="P+1" gate="1" x="-17.78" y="40.64" smashed="yes">
+<attribute name="VALUE" x="-20.32" y="35.56" size="1.778" layer="96" rot="R90"/>
+</instance>
+<instance part="C1" gate="G$1" x="20.32" y="-15.24" smashed="yes">
+<attribute name="NAME" x="21.844" y="-14.859" size="1.778" layer="95"/>
+<attribute name="VALUE" x="21.844" y="-19.939" size="1.778" layer="96"/>
+</instance>
+<instance part="C2" gate="G$1" x="40.64" y="-15.24" smashed="yes">
+<attribute name="NAME" x="42.164" y="-14.859" size="1.778" layer="95"/>
+<attribute name="VALUE" x="42.164" y="-19.939" size="1.778" layer="96"/>
+</instance>
+<instance part="C3" gate="G$1" x="30.48" y="7.62" smashed="yes">
+<attribute name="NAME" x="32.004" y="8.001" size="1.778" layer="95"/>
+<attribute name="VALUE" x="32.004" y="2.921" size="1.778" layer="96"/>
+</instance>
+<instance part="R1" gate="G$1" x="27.94" y="-25.4" smashed="yes">
+<attribute name="NAME" x="24.13" y="-24.0284" size="1.778" layer="95"/>
+<attribute name="VALUE" x="24.13" y="-28.321" size="1.778" layer="96"/>
+</instance>
+<instance part="R2" gate="G$1" x="27.94" y="-30.48" smashed="yes">
+<attribute name="NAME" x="24.13" y="-29.1084" size="1.778" layer="95"/>
+<attribute name="VALUE" x="24.13" y="-33.401" size="1.778" layer="96"/>
+</instance>
+<instance part="R3" gate="G$1" x="30.48" y="17.78" smashed="yes" rot="R90">
+<attribute name="NAME" x="29.1084" y="13.97" size="1.778" layer="95" rot="R90"/>
+<attribute name="VALUE" x="33.401" y="13.97" size="1.778" layer="96" rot="R90"/>
+</instance>
+<instance part="P+2" gate="1" x="30.48" y="25.4" smashed="yes">
+<attribute name="VALUE" x="27.94" y="20.32" size="1.778" layer="96" rot="R90"/>
+</instance>
+<instance part="GND1" gate="1" x="-22.86" y="-20.32" smashed="yes">
+<attribute name="VALUE" x="-25.4" y="-22.86" size="1.778" layer="96"/>
+</instance>
+<instance part="GND2" gate="1" x="-27.94" y="0" smashed="yes">
+<attribute name="VALUE" x="-30.48" y="-2.54" size="1.778" layer="96"/>
+</instance>
+<instance part="GND3" gate="1" x="40.64" y="-22.86" smashed="yes">
+<attribute name="VALUE" x="38.1" y="-25.4" size="1.778" layer="96"/>
+</instance>
+<instance part="GND4" gate="1" x="30.48" y="0" smashed="yes">
+<attribute name="VALUE" x="27.94" y="-2.54" size="1.778" layer="96"/>
+</instance>
+<instance part="C4" gate="G$1" x="-22.86" y="15.24" smashed="yes">
+<attribute name="NAME" x="-21.336" y="15.621" size="1.778" layer="95"/>
+<attribute name="VALUE" x="-21.336" y="10.541" size="1.778" layer="96"/>
+</instance>
+<instance part="R4" gate="G$1" x="-22.86" y="25.4" smashed="yes" rot="R90">
+<attribute name="NAME" x="-24.2316" y="21.59" size="1.778" layer="95" rot="R90"/>
+<attribute name="VALUE" x="-19.939" y="21.59" size="1.778" layer="96" rot="R90"/>
+</instance>
+<instance part="P+3" gate="1" x="-22.86" y="33.02" smashed="yes">
+<attribute name="VALUE" x="-25.4" y="27.94" size="1.778" layer="96" rot="R90"/>
+</instance>
+<instance part="GND5" gate="1" x="-22.86" y="7.62" smashed="yes">
+<attribute name="VALUE" x="-25.4" y="5.08" size="1.778" layer="96"/>
+</instance>
 </instances>
 <busses>
 </busses>
 <nets>
+<net name="+5V" class="0">
+<segment>
+<pinref part="P+2" gate="1" pin="+5V"/>
+<pinref part="R3" gate="G$1" pin="2"/>
+</segment>
+<segment>
+<pinref part="P+3" gate="1" pin="+5V"/>
+<pinref part="R4" gate="G$1" pin="2"/>
+</segment>
+</net>
+<net name="GND" class="0">
+<segment>
+<pinref part="GND4" gate="1" pin="GND"/>
+<pinref part="C3" gate="G$1" pin="2"/>
+</segment>
+<segment>
+<pinref part="GND3" gate="1" pin="GND"/>
+<pinref part="C2" gate="G$1" pin="2"/>
+</segment>
+<segment>
+<pinref part="U$1" gate="G$1" pin="VSS"/>
+<pinref part="GND2" gate="1" pin="GND"/>
+<wire x1="-15.24" y1="2.54" x2="-27.94" y2="2.54" width="0.1524" layer="91"/>
+</segment>
+<segment>
+<pinref part="GND5" gate="1" pin="GND"/>
+<pinref part="C4" gate="G$1" pin="2"/>
+</segment>
+</net>
+<net name="N$2" class="0">
+<segment>
+<pinref part="C3" gate="G$1" pin="1"/>
+<pinref part="R3" gate="G$1" pin="1"/>
+<wire x1="30.48" y1="12.7" x2="30.48" y2="10.16" width="0.1524" layer="91"/>
+<pinref part="U$1" gate="G$1" pin="CKIN"/>
+<wire x1="15.24" y1="7.62" x2="17.78" y2="7.62" width="0.1524" layer="91"/>
+<wire x1="17.78" y1="7.62" x2="17.78" y2="10.16" width="0.1524" layer="91"/>
+<wire x1="17.78" y1="10.16" x2="30.48" y2="10.16" width="0.1524" layer="91"/>
+<junction x="30.48" y="10.16"/>
+</segment>
+</net>
+<net name="N$1" class="0">
+<segment>
+<pinref part="U$1" gate="G$1" pin="GND"/>
+<wire x1="15.24" y1="-2.54" x2="40.64" y2="-2.54" width="0.1524" layer="91"/>
+<pinref part="C2" gate="G$1" pin="1"/>
+<wire x1="40.64" y1="-2.54" x2="40.64" y2="-12.7" width="0.1524" layer="91"/>
+</segment>
+</net>
+<net name="N$3" class="0">
+<segment>
+<pinref part="R2" gate="G$1" pin="1"/>
+<pinref part="C1" gate="G$1" pin="2"/>
+<wire x1="22.86" y1="-30.48" x2="20.32" y2="-30.48" width="0.1524" layer="91"/>
+<wire x1="20.32" y1="-30.48" x2="20.32" y2="-25.4" width="0.1524" layer="91"/>
+<pinref part="R1" gate="G$1" pin="1"/>
+<wire x1="20.32" y1="-25.4" x2="20.32" y2="-20.32" width="0.1524" layer="91"/>
+<wire x1="22.86" y1="-25.4" x2="20.32" y2="-25.4" width="0.1524" layer="91"/>
+<junction x="20.32" y="-25.4"/>
+</segment>
+</net>
+<net name="N$4" class="0">
+<segment>
+<pinref part="U$1" gate="G$1" pin="IN"/>
+<pinref part="C1" gate="G$1" pin="1"/>
+<wire x1="15.24" y1="-7.62" x2="20.32" y2="-7.62" width="0.1524" layer="91"/>
+<wire x1="20.32" y1="-7.62" x2="20.32" y2="-12.7" width="0.1524" layer="91"/>
+</segment>
+</net>
+<net name="N$5" class="0">
+<segment>
+<pinref part="C4" gate="G$1" pin="1"/>
+<pinref part="R4" gate="G$1" pin="1"/>
+<wire x1="-22.86" y1="20.32" x2="-22.86" y2="17.78" width="0.1524" layer="91"/>
+<pinref part="U$1" gate="G$1" pin="VDD"/>
+<wire x1="-15.24" y1="7.62" x2="-15.24" y2="17.78" width="0.1524" layer="91"/>
+<wire x1="-15.24" y1="17.78" x2="-22.86" y2="17.78" width="0.1524" layer="91"/>
+<junction x="-22.86" y="17.78"/>
+</segment>
+</net>
 </nets>
 </sheet>
@@
 </drawing>
 <compatibility>
+<note version="8.2" severity="warning">
+Since Version 8.2, EAGLE supports online libraries. The ids
+of those online libraries will not be understood (or retained)
+with this version.
+</note>
 <note version="8.3" severity="warning">
 Since Version 8.3, EAGLE supports URNs for individual library
@@
 will not be understood (or retained) with this version.
 </note>
+<note version="8.3" severity="warning">
+Since Version 8.3, EAGLE supports the association of 3D packages
+with devices in libraries, schematics, and board files. Those 3D
+packages will not be understood (or retained) with this version.
+</note>
 </compatibility>

Commit message: [add]基板作成
Changed lines of the file:
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@@
 </variantdefs>
 <classes>
-<class number="0" name="default" width="0" drill="0">
+<class number="0" name="default" width="1.27" drill="0">
+<clearance class="0" value="0.381"/>
 </class>
 </classes>
 <parts>
 <part name="U$1" library="ynakano1127" deviceset="MSGEQ7" device=""/>
-<part name="P+1" library="supply1" library_urn="urn:adsk.eagle:library:371" deviceset="+5V" device=""/>
 <part name="C1" library="capacitor-wima" library_urn="urn:adsk.eagle:library:116" deviceset="C" device="2.5/2" package3d_urn="urn:adsk.eagle:package:5415/1"/>
 <part name="C2" library="capacitor-wima" library_urn="urn:adsk.eagle:library:116" deviceset="C" device="2.5/2" package3d_urn="urn:adsk.eagle:package:5415/1"/>
@@
 <part name="R3" library="resistor-power" library_urn="urn:adsk.eagle:library:344" deviceset="R" device="AC01" package3d_urn="urn:adsk.eagle:package:25124/1"/>
 <part name="P+2" library="supply1" library_urn="urn:adsk.eagle:library:371" deviceset="+5V" device=""/>
-<part name="GND1" library="supply1" library_urn="urn:adsk.eagle:library:371" deviceset="GND" device=""/>
 <part name="GND2" library="supply1" library_urn="urn:adsk.eagle:library:371" deviceset="GND" device=""/>
 <part name="GND3" library="supply1" library_urn="urn:adsk.eagle:library:371" deviceset="GND" device=""/>
@@
 <instances>
 <instance part="U$1" gate="G$1" x="0" y="0" smashed="yes"/>
-<instance part="P+1" gate="1" x="-17.78" y="40.64" smashed="yes">
-<attribute name="VALUE" x="-20.32" y="35.56" size="1.778" layer="96" rot="R90"/>
-</instance>
 <instance part="C1" gate="G$1" x="20.32" y="-15.24" smashed="yes">
 <attribute name="NAME" x="21.844" y="-14.859" size="1.778" layer="95"/>
@@
 <attribute name="VALUE" x="27.94" y="20.32" size="1.778" layer="96" rot="R90"/>
 </instance>
-<instance part="GND1" gate="1" x="-22.86" y="-20.32" smashed="yes">
-<attribute name="VALUE" x="-25.4" y="-22.86" size="1.778" layer="96"/>
-</instance>
 <instance part="GND2" gate="1" x="-27.94" y="0" smashed="yes">
