File: Test.brd (EAGLE design)
At the start: 43.2 x 53 mm, 9 parts

Commit message: [add]値
Parts:
- removed R4: (no value), resistor-power:AC01
- C1: value (none) -> 0.01u
- C2, C4: value (none) -> 0.1u
- C3: value (none) -> 33p
- R1, R2, R3: value (none) -> 200k
Connections:
- removed net N$5: C4.1, R4.1, U$1.1
- net +5V: now also C4.1, U$1.1; no longer R4.2
Routing:
- net N$5: track 60.6 -> 0.00 mm
- net +5V: track 7.86 -> 19.8 mm
Changed lines of the file:
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@@
 </autorouter>
 <elements>
-<element name="C1" library="capacitor-wima" library_urn="urn:adsk.eagle:library:116" package="C2.5-2" package3d_urn="urn:adsk.eagle:package:5415/1" value="" x="10.16" y="24.13" smashed="yes" rot="R90">
+<element name="C1" library="capacitor-wima" library_urn="urn:adsk.eagle:library:116" package="C2.5-2" package3d_urn="urn:adsk.eagle:package:5415/1" value="0.01u" x="10.16" y="24.13" smashed="yes" rot="R90">
 <attribute name="NAME" x="8.636" y="22.479" size="1.27" layer="25" ratio="10" rot="R90"/>
 <attribute name="VALUE" x="12.954" y="22.479" size="1.27" layer="27" ratio="10" rot="R90"/>
 </element>
-<element name="C2" library="capacitor-wima" library_urn="urn:adsk.eagle:library:116" package="C2.5-2" package3d_urn="urn:adsk.eagle:package:5415/1" value="" x="5.08" y="21.59" smashed="yes" rot="R180">
+<element name="C2" library="capacitor-wima" library_urn="urn:adsk.eagle:library:116" package="C2.5-2" package3d_urn="urn:adsk.eagle:package:5415/1" value="0.1u" x="5.08" y="21.59" smashed="yes" rot="R180">
 <attribute name="NAME" x="6.731" y="20.066" size="1.27" layer="25" ratio="10" rot="R180"/>
 <attribute name="VALUE" x="6.731" y="24.384" size="1.27" layer="27" ratio="10" rot="R180"/>
 </element>
-<element name="C3" library="capacitor-wima" library_urn="urn:adsk.eagle:library:116" package="C2.5-2" package3d_urn="urn:adsk.eagle:package:5415/1" value="" x="27.94" y="46.99" smashed="yes">
+<element name="C3" library="capacitor-wima" library_urn="urn:adsk.eagle:library:116" package="C2.5-2" package3d_urn="urn:adsk.eagle:package:5415/1" value="33p" x="27.94" y="46.99" smashed="yes">
 <attribute name="NAME" x="26.289" y="48.514" size="1.27" layer="25" ratio="10"/>
 <attribute name="VALUE" x="26.289" y="44.196" size="1.27" layer="27" ratio="10"/>
 </element>
-<element name="C4" library="capacitor-wima" library_urn="urn:adsk.eagle:library:116" package="C2.5-2" package3d_urn="urn:adsk.eagle:package:5415/1" value="" x="5.08" y="46.99" smashed="yes" rot="R180">
+<element name="C4" library="capacitor-wima" library_urn="urn:adsk.eagle:library:116" package="C2.5-2" package3d_urn="urn:adsk.eagle:package:5415/1" value="0.1u" x="5.08" y="46.99" smashed="yes" rot="R180">
 <attribute name="NAME" x="6.731" y="45.466" size="1.27" layer="25" ratio="10" rot="R180"/>
 <attribute name="VALUE" x="6.731" y="49.784" size="1.27" layer="27" ratio="10" rot="R180"/>
 </element>
-<element name="R1" library="resistor-power" library_urn="urn:adsk.eagle:library:344" package="AC01" package3d_urn="urn:adsk.eagle:package:25124/1" value="" x="25.4" y="16.51" smashed="yes">
+<element name="R1" library="resistor-power" library_urn="urn:adsk.eagle:library:344" package="AC01" package3d_urn="urn:adsk.eagle:package:25124/1" value="200k" x="25.4" y="16.51" smashed="yes">
 <attribute name="MF" value="" x="48.26" y="2.54" size="1.778" layer="27" display="off"/>
 <attribute name="MPN" value="" x="48.26" y="2.54" size="1.778" layer="27" display="off"/>
@@
 <attribute name="VALUE" x="20.955" y="15.875" size="1.778" layer="27" ratio="10"/>
 </element>
-<element name="R2" library="resistor-power" library_urn="urn:adsk.eagle:library:344" package="AC01" package3d_urn="urn:adsk.eagle:package:25124/1" value="" x="25.4" y="24.13" smashed="yes">
+<element name="R2" library="resistor-power" library_urn="urn:adsk.eagle:library:344" package="AC01" package3d_urn="urn:adsk.eagle:package:25124/1" value="200k" x="25.4" y="24.13" smashed="yes">
 <attribute name="MF" value="" x="48.26" y="2.54" size="1.778" layer="27" display="off"/>
 <attribute name="MPN" value="" x="48.26" y="2.54" size="1.778" layer="27" display="off"/>
@@
 <attribute name="VALUE" x="20.955" y="23.495" size="1.778" layer="27" ratio="10"/>
 </element>
-<element name="R3" library="resistor-power" library_urn="urn:adsk.eagle:library:344" package="AC01" package3d_urn="urn:adsk.eagle:package:25124/1" value="" x="25.4" y="31.75" smashed="yes">
+<element name="R3" library="resistor-power" library_urn="urn:adsk.eagle:library:344" package="AC01" package3d_urn="urn:adsk.eagle:package:25124/1" value="200k" x="25.4" y="31.75" smashed="yes">
 <attribute name="MF" value="" x="48.26" y="2.54" size="1.778" layer="27" display="off"/>
 <attribute name="MPN" value="" x="48.26" y="2.54" size="1.778" layer="27" display="off"/>
@@
 <attribute name="OC_NEWARK" value="unknown" x="48.26" y="2.54" size="1.778" layer="27" display="off"/>
 <attribute name="VALUE" x="20.955" y="31.115" size="1.778" layer="27" ratio="10"/>
-</element>
-<element name="R4" library="resistor-power" library_urn="urn:adsk.eagle:library:344" package="AC01" package3d_urn="urn:adsk.eagle:package:25124/1" value="" x="25.4" y="39.37" smashed="yes">
-<attribute name="MF" value="" x="48.26" y="2.54" size="1.778" layer="27" display="off"/>
-<attribute name="MPN" value="" x="48.26" y="2.54" size="1.778" layer="27" display="off"/>
-<attribute name="NAME" x="19.685" y="41.91" size="1.778" layer="25" ratio="10"/>
-<attribute name="OC_FARNELL" value="unknown" x="48.26" y="2.54" size="1.778" layer="27" display="off"/>
-<attribute name="OC_NEWARK" value="unknown" x="48.26" y="2.54" size="1.778" layer="27" display="off"/>
-<attribute name="VALUE" x="20.955" y="38.735" size="1.778" layer="27" ratio="10"/>
 </element>
 <element name="U$1" library="SpectralAnalyzer" library_urn="urn:adsk.eagle:library:7692814" package="DIL08" package3d_urn="urn:adsk.eagle:package:7691021/2" value="MSGEQ7" x="7.62" y="-7.62" smashed="yes">
@@
 <signal name="+5V">
 <contactref element="R3" pad="2"/>
-<contactref element="R4" pad="2"/>
 <wire x1="34.671" y1="38.7985" x2="34.671" y2="32.1945" width="1.27" layer="16"/>
 <wire x1="34.671" y1="32.1945" x2="34.3" y2="31.75" width="1.27" layer="16"/>
-<wire x1="34.671" y1="38.7985" x2="34.3" y2="39.37" width="1.27" layer="16"/>
+<contactref element="C4" pad="1"/>
+<contactref element="U$1" pad="1"/>
+<wire x1="9.0805" y1="46.228" x2="6.604" y2="46.228" width="1.27" layer="16"/>
+<wire x1="15.6845" y1="39.624" x2="9.0805" y2="46.228" width="1.27" layer="16"/>
+<wire x1="6.604" y1="46.228" x2="6.35" y2="46.99" width="1.27" layer="16"/>
+<wire x1="15.6845" y1="39.624" x2="34.671" y2="38.7985" width="0" layer="19" extent="16-16"/>
+<wire x1="3.81" y1="-11.43" x2="15.6845" y2="39.624" width="0" layer="19" extent="16-16"/>
 </signal>
 <signal name="GND">
@@
 <wire x1="11.43" y1="-3.81" x2="24.765" y2="10.7315" width="0" layer="19" extent="16-16"/>
 </signal>
-<signal name="N$5">
-<contactref element="C4" pad="1"/>
-<contactref element="R4" pad="1"/>
-<wire x1="18.161" y1="4.1275" x2="18.161" y2="3.302" width="1.27" layer="16"/>
-<wire x1="21.463" y1="7.4295" x2="18.161" y2="4.1275" width="1.27" layer="16"/>
-<wire x1="26.416" y1="7.4295" x2="21.463" y2="7.4295" width="1.27" layer="16"/>
-<wire x1="27.2415" y1="8.255" x2="26.416" y2="7.4295" width="1.27" layer="16"/>
-<wire x1="27.2415" y1="28.067" x2="27.2415" y2="8.255" width="1.27" layer="16"/>
-<wire x1="16.51" y1="38.7985" x2="27.2415" y2="28.067" width="1.27" layer="16"/>
-<wire x1="16.51" y1="38.7985" x2="16.5" y2="39.37" width="1.27" layer="16"/>
-<wire x1="9.0805" y1="46.228" x2="6.604" y2="46.228" width="1.27" layer="16"/>
-<wire x1="15.6845" y1="39.624" x2="9.0805" y2="46.228" width="1.27" layer="16"/>
-<wire x1="6.604" y1="46.228" x2="6.35" y2="46.99" width="1.27" layer="16"/>
-<wire x1="15.6845" y1="39.624" x2="16.5" y2="39.37" width="1.27" layer="16"/>
-<contactref element="U$1" pad="1"/>
-<wire x1="3.81" y1="-11.43" x2="18.161" y2="3.302" width="0" layer="19" extent="16-16"/>
-</signal>
 <signal name="N$6">

Commit message: [add]LM3914
Parts:
- added R4, R5: (no value), resistor-power:AC01
- added U$2: LB10, SpectralAnalyzer:LB10
- added U$3: LM3914, SpectralAnalyzer:DIL18
Connections:
- new net +12V: U$3.3, U$3.9
- new net N$10: U$2.12, U$3.10
- new net N$11: U$2.13, U$3.11
- new net N$12: U$2.14, U$3.12
- new net N$13: U$2.15, U$3.13
- new net N$14: U$2.16, U$3.14
- new net N$15: U$2.17, U$3.15
- new net N$16: U$2.18, U$3.16
- new net N$17: U$2.19, U$3.17
- new net N$18: U$2.20, U$3.18
- new net N$19: R4.1, R5.2, U$3.8
- new net N$21: U$3.5
- new net N$22: R4.2, U$3.6, U$3.7
- new net N$5: U$1.3
- new net N$7: U$1.4
- new net N$8: U$1.7
- new net N$9: U$2.11, U$3.1
- net +5V: now also U$2.1, U$2.10, U$2.2, U$2.3, U$2.4, U$2.5, U$2.6, U$2.7, U$2.8, U$2.9
- net GND: now also R5.1, U$3.2, U$3.4
Changed lines of the file:
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@@
 <attribute name="VALUE" x="4.064" y="-8.255" size="1.27" layer="27" ratio="10"/>
+</element>
+<element name="U$2" library="SpectralAnalyzer" library_urn="urn:adsk.eagle:library:7692814" package="LB10" package3d_urn="urn:adsk.eagle:package:7691019/2" value="LB10" x="15.24" y="-22.86" smashed="yes">
+<attribute name="NAME" x="2.54" y="-17.145" size="1.27" layer="25" ratio="10"/>
+<attribute name="VALUE" x="11.43" y="-17.145" size="1.27" layer="27" ratio="10"/>
+</element>
+<element name="U$3" library="SpectralAnalyzer" library_urn="urn:adsk.eagle:library:7692814" package="DIL18" package3d_urn="urn:adsk.eagle:package:7691020/2" value="LM3914" x="15.24" y="-35.56" smashed="yes">
+<attribute name="NAME" x="3.556" y="-38.608" size="1.27" layer="25" ratio="10" rot="R90"/>
+<attribute name="VALUE" x="5.715" y="-36.195" size="1.27" layer="27" ratio="10"/>
+</element>
+<element name="R4" library="resistor-power" library_urn="urn:adsk.eagle:library:344" package="AC01" package3d_urn="urn:adsk.eagle:package:25124/1" value="" x="10.16" y="-48.26" smashed="yes">
+<attribute name="MF" value="" x="10.16" y="-48.26" size="1.778" layer="27" display="off"/>
+<attribute name="MPN" value="" x="10.16" y="-48.26" size="1.778" layer="27" display="off"/>
+<attribute name="NAME" x="4.445" y="-45.72" size="1.778" layer="25" ratio="10"/>
+<attribute name="OC_FARNELL" value="unknown" x="10.16" y="-48.26" size="1.778" layer="27" display="off"/>
+<attribute name="OC_NEWARK" value="unknown" x="10.16" y="-48.26" size="1.778" layer="27" display="off"/>
+<attribute name="VALUE" x="5.715" y="-48.895" size="1.778" layer="27" ratio="10"/>
+</element>
+<element name="R5" library="resistor-power" library_urn="urn:adsk.eagle:library:344" package="AC01" package3d_urn="urn:adsk.eagle:package:25124/1" value="" x="10.16" y="-55.88" smashed="yes">
+<attribute name="MF" value="" x="10.16" y="-55.88" size="1.778" layer="27" display="off"/>
+<attribute name="MPN" value="" x="10.16" y="-55.88" size="1.778" layer="27" display="off"/>
+<attribute name="NAME" x="4.445" y="-53.34" size="1.778" layer="25" ratio="10"/>
+<attribute name="OC_FARNELL" value="unknown" x="10.16" y="-55.88" size="1.778" layer="27" display="off"/>
+<attribute name="OC_NEWARK" value="unknown" x="10.16" y="-55.88" size="1.778" layer="27" display="off"/>
+<attribute name="VALUE" x="5.715" y="-56.515" size="1.778" layer="27" ratio="10"/>
 </element>
 </elements>
@@
 <wire x1="15.6845" y1="39.624" x2="9.0805" y2="46.228" width="1.27" layer="16"/>
 <wire x1="6.604" y1="46.228" x2="6.35" y2="46.99" width="1.27" layer="16"/>
+<contactref element="U$2" pad="5"/>
+<contactref element="U$2" pad="1"/>
+<contactref element="U$2" pad="2"/>
+<contactref element="U$2" pad="3"/>
+<contactref element="U$2" pad="4"/>
+<contactref element="U$2" pad="8"/>
+<contactref element="U$2" pad="9"/>
+<contactref element="U$2" pad="10"/>
+<contactref element="U$2" pad="6"/>
+<contactref element="U$2" pad="7"/>
 <wire x1="15.6845" y1="39.624" x2="34.671" y2="38.7985" width="0" layer="19" extent="16-16"/>
 <wire x1="3.81" y1="-11.43" x2="15.6845" y2="39.624" width="0" layer="19" extent="16-16"/>
+<wire x1="3.81" y1="-26.67" x2="3.81" y2="-11.43" width="0" layer="19" extent="1-1"/>
+<wire x1="6.35" y1="-26.67" x2="3.81" y2="-26.67" width="0" layer="19" extent="1-1"/>
+<wire x1="8.89" y1="-26.67" x2="6.35" y2="-26.67" width="0" layer="19" extent="1-1"/>
+<wire x1="11.43" y1="-26.67" x2="8.89" y2="-26.67" width="0" layer="19" extent="1-1"/>
+<wire x1="13.97" y1="-26.67" x2="11.43" y2="-26.67" width="0" layer="19" extent="1-1"/>
+<wire x1="16.51" y1="-26.67" x2="13.97" y2="-26.67" width="0" layer="19" extent="1-1"/>
+<wire x1="19.05" y1="-26.67" x2="16.51" y2="-26.67" width="0" layer="19" extent="1-1"/>
+<wire x1="21.59" y1="-26.67" x2="19.05" y2="-26.67" width="0" layer="19" extent="1-1"/>
+<wire x1="24.13" y1="-26.67" x2="21.59" y2="-26.67" width="0" layer="19" extent="1-1"/>
+<wire x1="26.67" y1="-26.67" x2="24.13" y2="-26.67" width="0" layer="19" extent="1-1"/>
 </signal>
 <signal name="GND">
@@
 <wire x1="4.1275" y1="47.0535" x2="3.81" y2="46.99" width="1.27" layer="16"/>
 <contactref element="U$1" pad="2"/>
-<wire x1="20.6375" y1="4.1275" x2="3.81" y2="21.59" width="0" layer="19" extent="16-16"/>
-<wire x1="6.35" y1="-11.43" x2="20.6375" y2="3.302" width="0" layer="19" extent="16-16"/>
+<contactref element="U$3" pad="2"/>
+<contactref element="U$3" pad="4"/>
+<contactref element="R5" pad="1"/>
+<wire x1="7.62" y1="-39.37" x2="1.26" y2="-55.88" width="0" layer="19" extent="1-1"/>
+<wire x1="12.7" y1="-39.37" x2="7.62" y2="-39.37" width="0" layer="19" extent="1-1"/>
+<wire x1="6.35" y1="-11.43" x2="7.62" y2="-39.37" width="0" layer="19" extent="1-1"/>
+<wire x1="20.6375" y1="3.302" x2="6.35" y2="-11.43" width="0" layer="19" extent="16-16"/>
+<wire x1="3.81" y1="21.59" x2="20.6375" y2="4.1275" width="0" layer="19" extent="16-16"/>
 </signal>
 <signal name="N$2">
@@
 </polygon>
 </signal>
+<signal name="N$5">
+<contactref element="U$1" pad="3"/>
+</signal>
+<signal name="N$7">
+<contactref element="U$1" pad="4"/>
+</signal>
+<signal name="N$8">
+<contactref element="U$1" pad="7"/>
+</signal>
+<signal name="N$9">
+<contactref element="U$2" pad="11"/>
+<contactref element="U$3" pad="1"/>
+<wire x1="26.67" y1="-19.05" x2="5.08" y2="-39.37" width="0" layer="19" extent="1-1"/>
+</signal>
+<signal name="N$10">
+<contactref element="U$2" pad="12"/>
+<contactref element="U$3" pad="10"/>
+<wire x1="25.4" y1="-31.75" x2="24.13" y2="-19.05" width="0" layer="19" extent="1-1"/>
+</signal>
+<signal name="N$11">
+<contactref element="U$2" pad="13"/>
+<contactref element="U$3" pad="11"/>
+<wire x1="21.59" y1="-19.05" x2="22.86" y2="-31.75" width="0" layer="19" extent="1-1"/>
+</signal>
+<signal name="N$12">
+<contactref element="U$2" pad="14"/>
+<contactref element="U$3" pad="12"/>
+<wire x1="19.05" y1="-19.05" x2="20.32" y2="-31.75" width="0" layer="19" extent="1-1"/>
+</signal>
+<signal name="N$13">
+<contactref element="U$2" pad="15"/>
+<contactref element="U$3" pad="13"/>
+<wire x1="16.51" y1="-19.05" x2="17.78" y2="-31.75" width="0" layer="19" extent="1-1"/>
+</signal>
+<signal name="N$14">
+<contactref element="U$2" pad="16"/>
+<contactref element="U$3" pad="14"/>
+<wire x1="13.97" y1="-19.05" x2="15.24" y2="-31.75" width="0" layer="19" extent="1-1"/>
+</signal>
+<signal name="N$15">
+<contactref element="U$2" pad="17"/>
+<contactref element="U$3" pad="15"/>
+<wire x1="11.43" y1="-19.05" x2="12.7" y2="-31.75" width="0" layer="19" extent="1-1"/>
+</signal>
+<signal name="N$16">
+<contactref element="U$2" pad="18"/>
+<contactref element="U$3" pad="16"/>
+<wire x1="8.89" y1="-19.05" x2="10.16" y2="-31.75" width="0" layer="19" extent="1-1"/>
+</signal>
+<signal name="N$17">
+<contactref element="U$2" pad="19"/>
+<contactref element="U$3" pad="17"/>
+<wire x1="6.35" y1="-19.05" x2="7.62" y2="-31.75" width="0" layer="19" extent="1-1"/>
+</signal>
+<signal name="N$18">
+<contactref element="U$2" pad="20"/>
+<contactref element="U$3" pad="18"/>
+<wire x1="3.81" y1="-19.05" x2="5.08" y2="-31.75" width="0" layer="19" extent="1-1"/>
+</signal>
+<signal name="+12V">
+<contactref element="U$3" pad="3"/>
+<contactref element="U$3" pad="9"/>
+<wire x1="25.4" y1="-39.37" x2="10.16" y2="-39.37" width="0" layer="19" extent="1-1"/>
+</signal>
+<signal name="N$21">
+<contactref element="U$3" pad="5"/>
+</signal>
+<signal name="N$22">
+<contactref element="U$3" pad="7"/>
+<contactref element="U$3" pad="6"/>
+<contactref element="R4" pad="2"/>
+<wire x1="17.78" y1="-39.37" x2="19.06" y2="-48.26" width="0" layer="19" extent="1-1"/>
+<wire x1="20.32" y1="-39.37" x2="17.78" y2="-39.37" width="0" layer="19" extent="1-1"/>
+</signal>
+<signal name="N$19">
+<contactref element="R4" pad="1"/>
+<contactref element="R5" pad="2"/>
+<contactref element="U$3" pad="8"/>
+<wire x1="19.06" y1="-55.88" x2="1.26" y2="-48.26" width="0" layer="19" extent="1-1"/>
+<wire x1="22.86" y1="-39.37" x2="19.06" y2="-55.88" width="0" layer="19" extent="1-1"/>
+</signal>
 </signals>
