File: Main.sch (EAGLE design)
At the start: 12 parts, among them IC1 LM358N, IC2 MSGEQ7DIL, T1 2SC1306, U1 ESP32-DEVKITC-32D

Commit message: [rm]いったん全部消去
Parts:
- removed C1: 33pF, eagle-ltspice:C
- removed C2: 0.01uF, eagle-ltspice:C
- removed C3: 0.1uF, eagle-ltspice:C
- removed IC1: LM358N, linear:LM358N
- removed IC2: MSGEQ7DIL, MSGEQ7:MSGEQ7DIL
- removed N1: IN-9, russian-nixies:IN-9
- removed R1: 300Ω, eagle-ltspice:R
- removed R2: 200kΩ, eagle-ltspice:R
- removed R3: (no value), 161104 Library by matsu:TRIM_EU-B25P
- removed R4: 22kΩ, eagle-ltspice:R
- removed T1: 2SC1306, transistor-neu-to92:2SC1306
- removed U1: ESP32-DEVKITC-32D, ESP32-DEVKITC-32D:ESP32-DEVKITC-32D
Connections:
- removed net +3V3: R4.2, U1.3V3
- removed net +5V: R3.E, U1.EXT_5V
- removed net GND: C1.2, C3.2, IC2.CG, R1.1, U1.GND3
- removed net N$1: IC1A.-IN, R1.2, T1.E
- removed net N$10: IC2.STROBE, U1.IO23
- removed net N$11: IC2.RESET, U1.IO22
- removed net N$2: IC2.AUDIO_IN, R3.A
- removed net N$3: IC1A.OUT, T1.B
- removed net N$4: N1.A, T1.C
- removed net N$5: C2.2, R3.S
- removed net N$6: C1.1, IC2.CKIN, R2.2
- removed net N$7: C2.1, R4.1
- removed net N$8: IC1A.+IN, IC2.DCOUT
- removed net N$9: C3.1, IC2.GND
- removed net V+: N1.K
- removed net VDD: R2.1

Commit message: [add]すべてを実装しなおした
Parts:
- added C1: 0.01u, SpectralAnalyzer:CAPACITOR
- added C2: 0.1u, SpectralAnalyzer:CAPACITOR
- added C3: 33p, SpectralAnalyzer:CAPACITOR
- added IC1: MSGEQ7, SpectralAnalyzer:MSGEQ7
- added IC2, IC3, IC4, IC5: LM358N, SpectralAnalyzer:LM358N
- added JP1, JP2: (no value), SpectralAnalyzer:PINHD-1X15
- added JP3, JP4, JP5, JP6, JP7: TERMINAL_BLOCK_2, SpectralAnalyzer:TERMINAL_BLOCK_2
- added R1, R2: 22k, SpectralAnalyzer:RESISTOR
- added R3: 200k, SpectralAnalyzer:RESISTOR
- added R4, R5, R6, R7, R8: 330, SpectralAnalyzer:RESISTOR
- added R9: 10k, SpectralAnalyzer:RK0972A103L15F
- added T1, T2, T3, T4, T5: 2SC3631, SpectralAnalyzer:2SC3631
- added U$1: DC_JACK, SpectralAnalyzer:DC_JACK
- added X1, X2: 3.3MM_AUDIO_JACK, SpectralAnalyzer:3.3MM_AUDIO_JACK
Connections:
- new net GND: C2.2, C3.2, IC1.VSS, IC2P.V-, IC3P.V-, IC4P.V-, IC5P.V-, JP1.2, R4.1, R5.1, R6.1, R7.1, R8.1, U$1.GND, X1.1
- new net N$1: C1.1, R1.2, R2.2
- new net N$10: JP1.8
- new net N$11: JP2.15
- new net N$12: JP2.14
- new net N$13: JP2.5
- new net N$14: JP2.3
- new net N$15: JP2.4
- new net N$16: JP2.6
- new net N$17: JP2.7
- new net N$18: JP3.2, T1.C
- new net N$19: IC2A.IN-, R4.2, T1.E
- new net N$2: IC5A.IN+, R1.1, X1.3
- new net N$20: IC2A.OUT, T1.B
- new net N$21: JP4.2, T2.C
- new net N$22: IC2A.IN+
- new net N$23: IC2B.IN-, R5.2, T2.E
- new net N$24: IC2B.OUT, T2.B
- new net N$25: IC2B.IN+
- new net N$26: JP5.2, T3.C
- new net N$27: IC3A.IN-, R6.2, T3.E
- new net N$28: IC3A.OUT, T3.B
- new net N$29: IC3A.IN+
- new net N$3: IC5B.IN+, R2.1, X1.2
- new net N$30: JP6.2, T4.C
- new net N$31: IC3B.IN-, R7.2, T4.E
- new net N$32: IC3B.OUT, T4.B
- new net N$33: IC3B.IN+
- new net N$34: JP7.2, T5.C
- new net N$35: IC4A.IN-, R8.2, T5.E
- new net N$36: IC4A.OUT, T5.B
- new net N$37: IC4A.IN+
- new net N$38: R9A.1
- new net N$39: IC5A.IN-, IC5A.OUT, X2.3
- new net N$4: C1.2, R9A.2
- new net N$40: IC1.GND
- new net N$42: IC5B.IN-, IC5B.OUT, X2.2
- new net N$5: IC1.IN
- new net N$6: IC1.OUT
- new net N$7: IC1.STROBE
- new net N$8: IC1.RESET
- new net N$9: C3.1, IC1.CKIN, R3.1
- new net VCC: C2.1, IC1.VDD, IC2P.V+, IC3P.V+, IC4P.V+, IC5P.V+, JP1.1, JP3.1, JP4.1, JP5.1, JP6.1, JP7.1, R3.2, U$1.PWR
Other:
- note added: "AUDIO_IN"
- note added: "CH1"
- note added: "CH2"
- note added: "CH3"
- note added: "CH4"
- note added: "CH5"
- note added: "MSGEQ7_OUT"
- note added: "RESET"
- note added: "STROBE"
