File: Main.sch (EAGLE design)
At the start: 32 parts, among them IC1 MSGEQ7, IC2 LM358N, IC3 LM358N, IC4 LM358N, IC5 LM358N, T1 2SC3631, T2 2SC3631, T3 2SC3631, T4 2SC3631, T5 2SC3631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

Commit message: [add]書き忘れ
Changed lines of the file:
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@@
 <part name="GND16" library="SpectralAnalyzer" library_urn="urn:adsk.eagle:library:7692814" deviceset="GND" device=""/>
 <part name="IC5" library="SpectralAnalyzer" library_urn="urn:adsk.eagle:library:7692814" deviceset="LM358N" device="" package3d_urn="urn:adsk.eagle:package:7691021/3"/>
-<part name="P+12" library="SpectralAnalyzer" library_urn="urn:adsk.eagle:library:7692814" deviceset="VCC" device=""/>
+<part name="P+12" library="SpectralAnalyzer" library_urn="urn:adsk.eagle:library:7692814" deviceset="VCC" device="" value="5V"/>
 <part name="GND15" library="SpectralAnalyzer" library_urn="urn:adsk.eagle:library:7692814" deviceset="GND" device=""/>
 <part name="X2" library="SpectralAnalyzer" library_urn="urn:adsk.eagle:library:7692814" deviceset="3.3MM_AUDIO_JACK" device="" package3d_urn="urn:adsk.eagle:package:8555/1"/>
